Commit message: Updated robot descriptions with Force and Torque feedback sensors
Co-Authored-By: Priyam Panchal <priyam.panchal.65@gmail.com>

File: iiwa_stack/iiwa_description/urdf/iiwa7.urdf.xacro (robot description, xacro)
@@ -4,14 +4,22 @@
   <xacro:include filename="$(find iiwa_description)/urdf/materials.xacro" />
   <!--Import the lbr iiwa macro -->
+  <!-- To import the floating spacecraft+iiwa -->
   <xacro:include filename="$(find iiwa_description)/urdf/iiwa7_withspacecraft.xacro"/>
+  <!-- To import the default iiwa -->
+  <!-- <xacro:include filename="$(find iiwa_description)/urdf/iiwa7.xacro"/> -->
+  <!-- To import the limp iiwa (TODO make limp iiwa urdf) -->
+  <!-- <xacro:include filename="$(find iiwa_description)/urdf/iiwa7_limp.xacro"/> -->
   <xacro:arg name="hardware_interface" default="PositionJointInterface"/>
   <xacro:arg name="robot_name" default="iiwa"/>
   <xacro:arg name="origin_xyz" default="0 0 0"/>
   <xacro:arg name="origin_rpy" default="0 0 0"/>
-  <!-- Fix to world just for testing -->
+  <!-- Uncomment this line for fixing the robot to the world. Commented by default to have the robot floating -->
   <!-- <link name="world"/> -->
   <!--iiwa-->
-  <xacro:iiwa7 hardware_interface="$(arg hardware_interface)" robot_name="$(arg robot_name)" parent="iiwa_link_0">
-    <origin xyz="$(arg origin_xyz)" rpy="$(arg origin_rpy)" />
+  <!-- <xacro:iiwa7 hardware_interface="$(arg hardware_interface)" robot_name="$(arg robot_name)" parent="world"> -->
+  <xacro:iiwa7 hardware_interface="$(arg hardware_interface)" robot_name="$(arg robot_name)" parent="world">
+  <!-- <xacro:iiwa7 robot_name="$(arg robot_name)" parent="iiwa_link_0"> -->
+  <!-- This changes where the robot is spawned -->
+    <origin xyz="0 0 1" rpy="0 0 0" />
   </xacro:iiwa7>
 </robot>

File: iiwa_stack/iiwa_description/urdf/iiwa7.xacro (robot description, xacro)
@@ -14,10 +14,91 @@
   <xacro:property name="max_velocity" value="10"/>
   <xacro:macro name="iiwa7" params="parent hardware_interface robot_name *origin">
+  <!-- Gazebo force/torque sensors at each joint -->
+  <gazebo reference="iiwa_joint_1">
+    <provideFeedback>true</provideFeedback>
+  </gazebo>
+  <gazebo>
+    <plugin name="ft_sensor" filename="libgazebo_ros_ft_sensor.so">
+        <updateRate>100.0</updateRate>
+        <topicName>ft_sensor1_topic</topicName>
+        <jointName>iiwa_joint_1</jointName>
+    </plugin>
+  </gazebo>
+  <gazebo reference="iiwa_joint_2">
+    <provideFeedback>true</provideFeedback>
+  </gazebo>
+  <gazebo>
+    <plugin name="ft_sensor" filename="libgazebo_ros_ft_sensor.so">
+        <updateRate>100.0</updateRate>
+        <topicName>ft_sensor2_topic</topicName>
+        <jointName>iiwa_joint_2</jointName>
+    </plugin>
+  </gazebo>
+  <gazebo reference="iiwa_joint_3">
+    <provideFeedback>true</provideFeedback>
+  </gazebo>
+  <gazebo>
+    <plugin name="ft_sensor" filename="libgazebo_ros_ft_sensor.so">
+        <updateRate>100.0</updateRate>
+        <topicName>ft_sensor3_topic</topicName>
+        <jointName>iiwa_joint_3</jointName>
+    </plugin>
+  </gazebo>
+  <gazebo reference="iiwa_joint_4">
+    <provideFeedback>true</provideFeedback>
+  </gazebo>
+  <gazebo>
+    <plugin name="ft_sensor" filename="libgazebo_ros_ft_sensor.so">
+        <updateRate>100.0</updateRate>
+        <topicName>ft_sensor4_topic</topicName>
+        <jointName>iiwa_joint_4</jointName>
+    </plugin>
+  </gazebo>
+  <gazebo reference="iiwa_joint_5">
+    <provideFeedback>true</provideFeedback>
+  </gazebo>
+  <gazebo>
+    <plugin name="ft_sensor" filename="libgazebo_ros_ft_sensor.so">
+        <updateRate>100.0</updateRate>
+        <topicName>ft_sensor5_topic</topicName>
+        <jointName>iiwa_joint_5</jointName>
+    </plugin>
+  </gazebo>
+  <gazebo reference="iiwa_joint_6">
+    <provideFeedback>true</provideFeedback>
+  </gazebo>
+  <gazebo>
+    <plugin name="ft_sensor" filename="libgazebo_ros_ft_sensor.so">
+        <updateRate>100.0</updateRate>
+        <topicName>ft_sensor6_topic</topicName>
+        <jointName>iiwa_joint_6</jointName>
+    </plugin>
+  </gazebo>
+  <gazebo reference="iiwa_joint_7">
+    <provideFeedback>true</provideFeedback>
+  </gazebo>
+  <gazebo>
+    <plugin name="ft_sensor" filename="libgazebo_ros_ft_sensor.so">
+        <updateRate>100.0</updateRate>
+        <topicName>ft_sensor7_topic</topicName>
+        <jointName>iiwa_joint_7</jointName>
+    </plugin>
+  </gazebo>
+<gazebo reference="world_iiwa_joint">
+    <provideFeedback>true</provideFeedback>
+  </gazebo>
+  <gazebo>
+    <plugin name="ft_sensor" filename="libgazebo_ros_ft_sensor.so">
+        <updateRate>100.0</updateRate>
+        <topicName>ft_sensor_topic</topicName>
+        <jointName>world_iiwa_joint</jointName>
+    </plugin>
+</gazebo>
     <!--joint between {parent} and link_0-->
-    <!-- <joint name="${parent}_${robot_name}_joint" type="fixed">
+    <joint name="${parent}_${robot_name}_joint" type="fixed">
       <xacro:insert_block name="origin"/>
       <parent link="${parent}"/>
       <child link="${robot_name}_link_0"/>
-    </joint> -->
+    </joint>
     <link name="${robot_name}_link_0">
       <inertial>
@@ -268,6 +349,6 @@
       <inertial>
         <origin xyz="0 0 0.02" rpy="0 0 0"/>
-        <mass value="100"/>
-        <!-- <mass value="3.129"/> -->
+        <!-- <mass value="100"/> -->
+        <mass value="3.129"/>
         <inertia ixx="0.01464"  ixy="0.0005912"  ixz="0" iyy="0.01465" iyz="0" izz="0.002872" />
       </inertial>

File: iiwa_stack/iiwa_description/urdf/iiwa7_limp.xacro (robot description, xacro)
@@ -3,95 +3,8 @@
   <!-- Import all Gazebo-customization elements, including Gazebo colors -->
   <xacro:include filename="$(find iiwa_description)/urdf/iiwa.gazebo.xacro" />
-  <!-- Import Transmissions -->
-  <xacro:include filename="$(find iiwa_description)/urdf/iiwa.transmission.xacro" />
   <!-- Include Utilities -->
   <xacro:include filename="$(find iiwa_description)/urdf/utilities.xacro" />
-  <gazebo reference="">
-    <provideFeedback>true</provideFeedback>
-  </gazebo>
-  <gazebo>
-    <plugin name="ft_sensor" filename="libgazebo_ros_ft_sensor.so">
-        <updateRate>100.0</updateRate>
-        <topicName>ft_sensor0_topic</topicName>
-        <jointName></jointName>
-    </plugin>
-</gazebo>
-<gazebo reference="iiwa_joint_1">
-    <provideFeedback>true</provideFeedback>
-  </gazebo>
-  <gazebo>
-    <plugin name="ft_sensor" filename="libgazebo_ros_ft_sensor.so">
-        <updateRate>100.0</updateRate>
-        <topicName>ft_sensor1_topic</topicName>
-        <jointName>iiwa_joint_1</jointName>
-    </plugin>
-</gazebo>
-<gazebo reference="iiwa_joint_2">
-    <provideFeedback>true</provideFeedback>
-  </gazebo>
-  <gazebo>
-    <plugin name="ft_sensor" filename="libgazebo_ros_ft_sensor.so">
-        <updateRate>100.0</updateRate>
-        <topicName>ft_sensor2_topic</topicName>
-        <jointName>iiwa_joint_2</jointName>
-    </plugin>
-</gazebo>
-<gazebo reference="iiwa_joint_3">
-    <provideFeedback>true</provideFeedback>
-  </gazebo>
-  <gazebo>
-    <plugin name="ft_sensor" filename="libgazebo_ros_ft_sensor.so">
-        <updateRate>100.0</updateRate>
-        <topicName>ft_sensor3_topic</topicName>
-        <jointName>iiwa_joint_3</jointName>
-    </plugin>
-</gazebo>
-<gazebo reference="iiwa_joint_4">
-    <provideFeedback>true</provideFeedback>
-  </gazebo>
-  <gazebo>
-    <plugin name="ft_sensor" filename="libgazebo_ros_ft_sensor.so">
-        <updateRate>100.0</updateRate>
-        <topicName>ft_sensor4_topic</topicName>
-        <jointName>iiwa_joint_4</jointName>
-    </plugin>
-</gazebo>
-<gazebo reference="iiwa_joint_5">
-    <provideFeedback>true</provideFeedback>
-  </gazebo>
-  <gazebo>
-    <plugin name="ft_sensor" filename="libgazebo_ros_ft_sensor.so">
-        <updateRate>100.0</updateRate>
-        <topicName>ft_sensor5_topic</topicName>
-        <jointName>iiwa_joint_5</jointName>
-    </plugin>
-</gazebo>
-<gazebo reference="iiwa_joint_6">
-    <provideFeedback>true</provideFeedback>
-  </gazebo>
-  <gazebo>
-    <plugin name="ft_sensor" filename="libgazebo_ros_ft_sensor.so">
-        <updateRate>100.0</updateRate>
-        <topicName>ft_sensor6_topic</topicName>
-        <jointName>iiwa_joint_6</jointName>
-    </plugin>
-</gazebo>
-<gazebo reference="iiwa_joint_7">
-    <provideFeedback>true</provideFeedback>
-  </gazebo>
-  <gazebo>
-    <plugin name="ft_sensor" filename="libgazebo_ros_ft_sensor.so">
-        <updateRate>100.0</updateRate>
-        <topicName>ft_sensor7_topic</topicName>
-        <jointName>iiwa_joint_7</jointName>
-    </plugin>
-</gazebo>
   <!-- some constants -->
-  <xacro:property name="safety_controller_k_pos" value="100" />
-  <xacro:property name="safety_controller_k_vel" value="2" />
-  <xacro:property name="joint_damping" value="0.05" />
-  <xacro:property name="max_effort" value="300"/>
-  <xacro:property name="max_velocity" value="10"/>
-  <xacro:macro name="iiwa7" params="parent hardware_interface robot_name *origin">
+  <xacro:macro name="iiwa7" params="parent robot_name *origin">
     <!--joint between {parent} and link_0-->
     <!-- <joint name="${parent}_${robot_name}_joint" type="fixed">
@@ -134,5 +47,5 @@
     </joint>
     <link name="${robot_name}_link_0">
-      <inertial>${robot_name}_joint_1
+      <inertial>
         <origin xyz="-0.1 0 0.07" rpy="0 0 0"/>
         <mass value="5"/>
@@ -166,11 +79,4 @@
       <origin xyz="0 0 0.15" rpy="0 0 0"/>
       <axis xyz="0 0 1"/>
-      <limit lower="${-170 * PI / 180}" upper="${170 * PI / 180}"
-             effort="${max_effort}" velocity="${max_velocity}" />
-      <safety_controller soft_lower_limit="${-168 * PI / 180}"
-                         soft_upper_limit="${168 * PI / 180}"
-                         k_position="${safety_controller_k_pos}"
-                         k_velocity="${safety_controller_k_vel}"/>
-      <dynamics damping="${joint_damping}"/>
     </joint>
     <link name="${robot_name}_link_1">
@@ -200,11 +106,4 @@
       <origin xyz="0 0 0.19" rpy="${PI / 2}   0 ${PI}"/>
       <axis xyz="0 0 1"/>
-      <limit lower="${-120 * PI / 180}" upper="${120 * PI / 180}"
-             effort="${max_effort}" velocity="${max_velocity}" />
-      <safety_controller soft_lower_limit="${-118 * PI / 180}"
-                         soft_upper_limit="${118 * PI / 180}"
-                         k_position="${safety_controller_k_pos}"
-                         k_velocity="${safety_controller_k_vel}"/>
-      <dynamics damping="${joint_damping}"/>
     </joint>
     <link name="${robot_name}_link_2">
@@ -234,11 +133,4 @@
       <origin xyz="0 0.21 0" rpy="${PI / 2} 0 ${PI}"/>
       <axis xyz="0 0 1"/>
-      <limit lower="${-170 * PI / 180}" upper="${170 * PI / 180}"
-             effort="${max_effort}" velocity="${max_velocity}" />
-      <safety_controller soft_lower_limit="${-168 * PI / 180}"
-                         soft_upper_limit="${168 * PI / 180}"
-                         k_position="${safety_controller_k_pos}"
-                         k_velocity="${safety_controller_k_vel}"/>
-      <dynamics damping="${joint_damping}"/>
     </joint>
     <link name="${robot_name}_link_3">
@@ -268,11 +160,4 @@
       <origin xyz="0 0 0.19" rpy="${PI / 2} 0 0"/>
       <axis xyz="0 0 1"/>
-      <limit lower="${-120 * PI / 180}" upper="${120 * PI / 180}"
-             effort="${max_effort}" velocity="${max_velocity}" />
-      <safety_controller soft_lower_limit="${-118 * PI / 180}"
-                         soft_upper_limit="${118 * PI / 180}"
-                         k_position="${safety_controller_k_pos}"
-                         k_velocity="${safety_controller_k_vel}"/>
-      <dynamics damping="${joint_damping}"/>
     </joint>
     <link name="${robot_name}_link_4">
@@ -302,11 +187,4 @@
       <origin xyz="0 0.21 0" rpy="${-PI / 2} ${PI} 0"/>
       <axis xyz="0 0 1"/>
-      <limit lower="${-170 * PI / 180}" upper="${170 * PI / 180}"
-             effort="${max_effort}" velocity="${max_velocity}" />
-      <safety_controller soft_lower_limit="${-168 * PI / 180}"
-                         soft_upper_limit="${168 * PI / 180}"
-                         k_position="${safety_controller_k_pos}"
-                         k_velocity="${safety_controller_k_vel}"/>
-      <dynamics damping="${joint_damping}"/>
     </joint>
     <link name="${robot_name}_link_5">
@@ -336,11 +214,4 @@
       <origin xyz="0 0.06070 0.19" rpy="${PI / 2} 0 0"/>
       <axis xyz="0 0 1"/>
-      <limit lower="${-120 * PI / 180}" upper="${120 * PI / 180}"
-             effort="${max_effort}" velocity="${max_velocity}" />
-      <safety_controller soft_lower_limit="${-118 * PI / 180}"
-                         soft_upper_limit="${118 * PI / 180}"
-                         k_position="${safety_controller_k_pos}"
-                         k_velocity="${safety_controller_k_vel}"/>
-      <dynamics damping="${joint_damping}"/>
     </joint>
     <link name="${robot_name}_link_6">
@@ -370,11 +241,4 @@
       <origin xyz="0 0.081 0.06070" rpy="${- PI / 2} ${PI} 0"/>
       <axis xyz="0 0 1"/>
-      <limit lower="${-175 * PI / 180}" upper="${175 * PI / 180}"
-             effort="${max_effort}" velocity="${max_velocity}" />
-      <safety_controller soft_lower_limit="${-173 * PI / 180}"
-                         soft_upper_limit="${173 * PI / 180}"
-                         k_position="${safety_controller_k_pos}"
-                         k_velocity="${safety_controller_k_vel}"/>
-      <dynamics damping="${joint_damping}"/>
     </joint>
     <link name="${robot_name}_link_7">
@@ -408,6 +272,6 @@
     </link>
     <!--Extensions -->
-    <xacro:iiwa_gazebo robot_name="${robot_name}" />
-    <xacro:iiwa_transmission hardware_interface="${hardware_interface}"/>
+    <!-- <xacro:iiwa_gazebo robot_name="${robot_name}" /> -->
+    <!-- <xacro:iiwa_transmission hardware_interface="${hardware_interface}"/> -->
   </xacro:macro>
 </robot>
